File: schematics/schematics.kicad_sch (KiCad schematic)
At the start: 0 parts

Commit message: Hardware Side Done
Parts:
- added A1: Arduino_Nano_ESP32, Module:Arduino_Nano, symbol MCU_Module:Arduino_Nano_ESP32
- added U1, U2: MPU-6050, Sensor_Motion:InvenSense_QFN-24_4x4mm_P0.5mm, symbol Sensor_Motion:MPU-6050
Connections:
- new net GND: A1.29 (GND), A1.4 (GND), U1.18 (GND), U1.9 (AD0), U2.18 (GND)
- new net SCL: A1.24 (SCL/A5), U1.23 (SCL), U2.23 (SCL)
- new net SDA: A1.23 (SDA/A4), U1.24 (SDA), U2.24 (SDA)
- new net VDD: A1.17 (3V3), U1.13 (VDD), U2.13 (VDD), U2.9 (AD0)
- no-connect marks 0 -> 16
Other:
- note added: "FOREARM IMU"
- note added: "UPPERARM IMU"
